File: Hardware/Gameling.sch (KiCad schematic (older format))
At the start: 45 parts, among them J1 Conn_ARM_JTAG_SWD_10, Q1 BC817, SW1 SW_Push_LED, SW10 SW_Push_LED, SW11 SW_Push_LED, SW12 SW_Push_LED, SW13 SW_SPDT, SW2 SW_Push_LED, SW3 SW_Push_LED, SW4 SW_Push_LED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

Commit message: Update to new symbol and footprints libraries
Parts:
- BT1: footprint My_Library:BatteryHolder_Keystone_2468_2xAAA_NoSilkscreen -> my-footprints-library:BatteryHolder_Keystone_2468_2xAAA_NoSilkscreen
- BZ1: footprint My_Library:Buzzer_CUI_CPT-9019S-SMT_With3DModel -> my-footprints-library:Buzzer_CUI_CPT-9019S-SMT_With3DModel
- D1, D2, D3, D4: footprint My_Library:D_0805_2012Metric_Pad1.15x1.40mm_HandSolder_NoSilkscreen -> my-footprints-library:D_0805_2012Metric_Pad1.15x1.40mm_HandSolder_NoSilkscreen
- J1: footprint My_Library:Amphenol_FCI_ShroudedSocket_2x05_P1.27mm_Vertical_SMD -> my-footprints-library:Amphenol_FCI_ShroudedSocket_2x05_P1.27mm_Vertical_SMD
- L1: footprint My_Library:L_Bourns-SRN4018_With3DModel -> my-footprints-library:L_Bourns-SRN4018_With3DModel
- SW1, SW10, SW11, SW12, SW2, SW3, SW4, SW5, SW6, SW7, SW8, SW9: footprint My_Library:Generic_LED_Tactile_Button -> my-footprints-library:Generic_LED_Tactile_Button
- SW13: footprint My_Library:SW_CuK_OS102011MA1QN1_SPDT_Angled_With3DModel_NoSilkscreen -> my-footprints-library:SW_CuK_OS102011MA1QN1_SPDT_Angled_With3DModel_NoSilkscreen
- U1: footprint Nokia_5110-3310_LCD:Nokia_5110-3310_LCD_NoSilkscreen -> my-footprints-library:Nokia_5110-3310_LCD_NoSilkscreen; symbol Nokia_5110-3310_LCD:Nokia_5110_LCD -> my-symbols-library:Nokia_5110_LCD
- U3: symbol My_Symbol_Library:STM32L412KB -> my-symbols-library:STM32L412KB
- U4: symbol My_Symbol_Library:TPS27081A -> my-symbols-library:TPS27081A
- U5: symbol My_Symbol_Library:AAT1217 -> my-symbols-library:AAT1217
Changed lines of the file:
@@
 EESchema Schematic File Version 4
-LIBS:Gameling-cache
-EELAYER 29 0
+EELAYER 30 0
 EELAYER END
 $Descr A3 16535 11693
@@
 $EndDescr
 $Comp
-L My_Symbol_Library:STM32L412KB U3
+L my-symbols-library:STM32L412KB U3
 U 1 1 5D3D757F
 P 4400 9200
@@
 F 0 "BT1" H 9758 2346 50  0000 L CNN
 F 1 "Battery" H 9758 2255 50  0000 L CNN
-F 2 "My_Library:BatteryHolder_Keystone_2468_2xAAA_NoSilkscreen" V 9650 2360 50  0001 C CNN
+F 2 "my-footprints-library:BatteryHolder_Keystone_2468_2xAAA_NoSilkscreen" V 9650 2360 50  0001 C CNN
 F 3 "~" V 9650 2360 50  0001 C CNN
 	1    9650 2300
@@
 F 0 "SW13" H 10050 2185 50  0000 C CNN
 F 1 "SW_SPDT" H 10050 2094 50  0000 C CNN
-F 2 "My_Library:SW_CuK_OS102011MA1QN1_SPDT_Angled_With3DModel_NoSilkscreen" H 10050 1900 50  0001 C CNN
+F 2 "my-footprints-library:SW_CuK_OS102011MA1QN1_SPDT_Angled_With3DModel_NoSilkscreen" H 10050 1900 50  0001 C CNN
 F 3 "~" H 10050 1900 50  0001 C CNN
 	1    10050 1900
@@
 F 0 "L1" V 12919 1600 50  0000 C CNN
 F 1 "4.7uH" V 13010 1600 50  0000 C CNN
-F 2 "My_Library:L_Bourns-SRN4018_With3DModel" H 13100 1600 50  0001 C CNN
+F 2 "my-footprints-library:L_Bourns-SRN4018_With3DModel" H 13100 1600 50  0001 C CNN
 F 3 "~" H 13100 1600 50  0001 C CNN
 	1    13100 1600
@@
 $EndComp
 $Comp
-L My_Symbol_Library:AAT1217 U5
+L my-symbols-library:AAT1217 U5
 U 1 1 5D45AD20
 P 13750 1750
@@
 $EndComp
 $Comp
-L My_Symbol_Library:TPS27081A U4
+L my-symbols-library:TPS27081A U4
 U 1 1 5D45E6FD
 P 11200 2000
@@
 F 0 "J1" H 8257 9296 50  0000 R CNN
 F 1 "Conn_ARM_JTAG_SWD_10" H 8257 9205 50  0000 R CNN
-F 2 "My_Library:Amphenol_FCI_ShroudedSocket_2x05_P1.27mm_Vertical_SMD" H 8700 9250 50  0001 C CNN
+F 2 "my-footprints-library:Amphenol_FCI_ShroudedSocket_2x05_P1.27mm_Vertical_SMD" H 8700 9250 50  0001 C CNN
 F 3 "http://infocenter.arm.com/help/topic/com.arm.doc.ddi0314h/DDI0314H_coresight_components_trm.pdf" V 8350 8000 50  0001 C CNN
 	1    8700 9250
@@
 F 0 "BZ1" H 14202 5179 50  0000 L CNN
 F 1 "Buzzer" H 14202 5088 50  0000 L CNN
-F 2 "My_Library:Buzzer_CUI_CPT-9019S-SMT_With3DModel" V 14025 5250 50  0001 C CNN
+F 2 "my-footprints-library:Buzzer_CUI_CPT-9019S-SMT_With3DModel" V 14025 5250 50  0001 C CNN
 F 3 "~" V 14025 5250 50  0001 C CNN
 	1    14050 5150
@@
 F 0 "SW12" H 8450 6985 50  0000 C CNN
 F 1 "SW_Push_LED" H 8450 6894 50  0000 C CNN
-F 2 "My_Library:Generic_LED_Tactile_Button" H 8450 6900 50  0001 C CNN
+F 2 "my-footprints-library:Generic_LED_Tactile_Button" H 8450 6900 50  0001 C CNN
 F 3 "~" H 8450 6900 50  0001 C CNN
 	1    8450 6600
@@
 F 0 "SW8" H 7200 6335 50  0000 C CNN
 F 1 "SW_Push_LED" H 7200 6244 50  0000 C CNN
-F 2 "My_Library:Generic_LED_Tactile_Button" H 7200 6250 50  0001 C CNN
+F 2 "my-footprints-library:Generic_LED_Tactile_Button" H 7200 6250 50  0001 C CNN
 F 3 "~" H 7200 6250 50  0001 C CNN
 	1    7200 5950
@@
 F 0 "SW4" H 5950 5685 50  0000 C CNN
 F 1 "SW_Push_LED" H 5950 5594 50  0000 C CNN
-F 2 "My_Library:Generic_LED_Tactile_Button" H 5950 5600 50  0001 C CNN
+F 2 "my-footprints-library:Generic_LED_Tactile_Button" H 5950 5600 50  0001 C CNN
 F 3 "~" H 5950 5600 50  0001 C CNN
 	1    5950 5300
@@
 F 0 "SW11" H 7200 6985 50  0000 C CNN
 F 1 "SW_Push_LED" H 7200 6894 50  0000 C CNN
-F 2 "My_Library:Generic_LED_Tactile_Button" H 7200 6900 50  0001 C CNN
+F 2 "my-footprints-library:Generic_LED_Tactile_Button" H 7200 6900 50  0001 C CNN
 F 3 "~" H 7200 6900 50  0001 C CNN
 	1    7200 6600
@@
 F 0 "SW7" H 5950 6335 50  0000 C CNN
 F 1 "SW_Push_LED" H 5950 6244 50  0000 C CNN
-F 2 "My_Library:Generic_LED_Tactile_Button" H 5950 6250 50  0001 C CNN
+F 2 "my-footprints-library:Generic_LED_Tactile_Button" H 5950 6250 50  0001 C CNN
 F 3 "~" H 5950 6250 50  0001 C CNN
 	1    5950 5950
@@
 F 0 "SW3" H 8450 5085 50  0000 C CNN
 F 1 "SW_Push_LED" H 8450 4994 50  0000 C CNN
-F 2 "My_Library:Generic_LED_Tactile_Button" H 8450 5000 50  0001 C CNN
+F 2 "my-footprints-library:Generic_LED_Tactile_Button" H 8450 5000 50  0001 C CNN
 F 3 "~" H 8450 5000 50  0001 C CNN
 	1    8450 4700
@@
 F 0 "SW10" H 5950 6985 50  0000 C CNN
 F 1 "SW_Push_LED" H 5950 6894 50  0000 C CNN
-F 2 "My_Library:Generic_LED_Tactile_Button" H 5950 6900 50  0001 C CNN
+F 2 "my-footprints-library:Generic_LED_Tactile_Button" H 5950 6900 50  0001 C CNN
 F 3 "~" H 5950 6900 50  0001 C CNN
 	1    5950 6600
@@
 F 0 "SW6" H 8450 5685 50  0000 C CNN
 F 1 "SW_Push_LED" H 8450 5594 50  0000 C CNN
-F 2 "My_Library:Generic_LED_Tactile_Button" H 8450 5600 50  0001 C CNN
+F 2 "my-footprints-library:Generic_LED_Tactile_Button" H 8450 5600 50  0001 C CNN
 F 3 "~" H 8450 5600 50  0001 C CNN
 	1    8450 5300
@@
 F 0 "SW2" H 7200 5085 50  0000 C CNN
 F 1 "SW_Push_LED" H 7200 4994 50  0000 C CNN
-F 2 "My_Library:Generic_LED_Tactile_Button" H 7200 5000 50  0001 C CNN
+F 2 "my-footprints-library:Generic_LED_Tactile_Button" H 7200 5000 50  0001 C CNN
 F 3 "~" H 7200 5000 50  0001 C CNN
 	1    7200 4700
@@
 F 0 "SW9" H 8450 6335 50  0000 C CNN
 F 1 "SW_Push_LED" H 8450 6244 50  0000 C CNN
-F 2 "My_Library:Generic_LED_Tactile_Button" H 8450 6250 50  0001 C CNN
+F 2 "my-footprints-library:Generic_LED_Tactile_Button" H 8450 6250 50  0001 C CNN
 F 3 "~" H 8450 6250 50  0001 C CNN
 	1    8450 5950
@@
 F 0 "SW5" H 7200 5685 50  0000 C CNN
 F 1 "SW_Push_LED" H 7200 5594 50  0000 C CNN
-F 2 "My_Library:Generic_LED_Tactile_Button" H 7200 5600 50  0001 C CNN
+F 2 "my-footprints-library:Generic_LED_Tactile_Button" H 7200 5600 50  0001 C CNN
 F 3 "~" H 7200 5600 50  0001 C CNN
 	1    7200 5300
@@
 F 0 "SW1" H 5950 5085 50  0000 C CNN
 F 1 "SW_Push_LED" H 5950 4994 50  0000 C CNN
-F 2 "My_Library:Generic_LED_Tactile_Button" H 5950 5000 50  0001 C CNN
+F 2 "my-footprints-library:Generic_LED_Tactile_Button" H 5950 5000 50  0001 C CNN
 F 3 "~" H 5950 5000 50  0001 C CNN
 	1    5950 4700
@@
 F 0 "D2" H 1843 2666 50  0000 C CNN
 F 1 "LED" H 1843 2575 50  0000 C CNN
-F 2 "My_Library:D_0805_2012Metric_Pad1.15x1.40mm_HandSolder_NoSilkscreen" H 1850 2450 50  0001 C CNN
+F 2 "my-footprints-library:D_0805_2012Metric_Pad1.15x1.40mm_HandSolder_NoSilkscreen" H 1850 2450 50  0001 C CNN
 F 3 "~" H 1850 2450 50  0001 C CNN
 	1    1850 2450
@@
 F 0 "D4" H 3093 2666 50  0000 C CNN
 F 1 "LED" H 3093 2575 50  0000 C CNN
-F 2 "My_Library:D_0805_2012Metric_Pad1.15x1.40mm_HandSolder_NoSilkscreen" H 3100 2450 50  0001 C CNN
+F 2 "my-footprints-library:D_0805_2012Metric_Pad1.15x1.40mm_HandSolder_NoSilkscreen" H 3100 2450 50  0001 C CNN
 F 3 "~" H 3100 2450 50  0001 C CNN
 	1    3100 2450
@@
 F 0 "D3" H 3093 2316 50  0000 C CNN
 F 1 "LED" H 3093 2225 50  0000 C CNN
-F 2 "My_Library:D_0805_2012Metric_Pad1.15x1.40mm_HandSolder_NoSilkscreen" H 3100 2100 50  0001 C CNN
+F 2 "my-footprints-library:D_0805_2012Metric_Pad1.15x1.40mm_HandSolder_NoSilkscreen" H 3100 2100 50  0001 C CNN
 F 3 "~" H 3100 2100 50  0001 C CNN
 	1    3100 2100
@@
 F 0 "D1" H 1843 2316 50  0000 C CNN
 F 1 "LED" H 1843 2225 50  0000 C CNN
-F 2 "My_Library:D_0805_2012Metric_Pad1.15x1.40mm_HandSolder_NoSilkscreen" H 1850 2100 50  0001 C CNN
+F 2 "my-footprints-library:D_0805_2012Metric_Pad1.15x1.40mm_HandSolder_NoSilkscreen" H 1850 2100 50  0001 C CNN
 F 3 "~" H 1850 2100 50  0001 C CNN
 	1    1850 2100
@@
 $EndComp
 $Comp
-L Nokia_5110-3310_LCD:Nokia_5110_LCD U1
+L my-symbols-library:Nokia_5110_LCD U1
 U 1 1 5D3A64A5
 P 5950 2100
 F 0 "U1" H 6128 2158 60  0000 L CNN
 F 1 "Nokia_5110_LCD" H 6128 2052 60  0000 L CNN
-F 2 "Nokia_5110-3310_LCD:Nokia_5110-3310_LCD_NoSilkscreen" H 5950 2100 60  0001 C CNN
+F 2 "my-footprints-library:Nokia_5110-3310_LCD_NoSilkscreen" H 5950 2100 60  0001 C CNN
 F 3 "" H 5950 2100 60  0000 C CNN
 	1    5950 2100
